File: DroneBoard/hardware/DroneCarrier/_autosave-cm4-gpio.kicad_sch (KiCad schematic)
At the start: 21 parts, among them J3 Conn_02x07_Odd_Even, J3 DNP, J4 Conn_01x03, J5 Conn_01x03, J6 Conn_01x03, J7 Micro_SD_Card_Det, U4 74LVC1G07SE-7, U5 74LVC1G07SE-7

Commit message: Labelling needs to be compared to the RPi CM4
Connections:
- no-connect marks 1 -> 14
Changed lines of the file:
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@@
   (junction (at 209.55 119.38) (diameter 1.016) (color 0 0 0 0))
   (junction (at 260.35 76.2) (diameter 1.016) (color 0 0 0 0))
+  (no_connect (at 41.91 22.86))
+  (no_connect (at 41.91 25.4))
+  (no_connect (at 41.91 30.48))
+  (no_connect (at 41.91 33.02))
+  (no_connect (at 41.91 38.1))
+  (no_connect (at 41.91 40.64))
+  (no_connect (at 102.87 22.86))
+  (no_connect (at 102.87 25.4))
+  (no_connect (at 102.87 30.48))
+  (no_connect (at 102.87 33.02))
+  (no_connect (at 102.87 38.1))
+  (no_connect (at 102.87 40.64))
+  (no_connect (at 102.87 43.18))
   (no_connect (at 242.57 147.32))
   (wire (pts (xy 13.97 170.18) (xy 27.94 170.18))
